File: design.kicad_sch (KiCad schematic)
At the start: 0 parts

Commit message: first commit
Parts:
- added C1, C10, C6: 10uF, Capacitor_SMD:C_0805_2012Metric, symbol Device:C_Small
- added C11, C3, C7, C? (x2): 1uF, Capacitor_SMD:C_0805_2012Metric, symbol Device:C_Small
- added C2, C5, C9: 0.1uF, Capacitor_SMD:C_0805_2012Metric, symbol Device:C_Small
- added C4, C8: 120uF, Capacitor_THT:CP_Radial_D8.0mm_P5.00mm, symbol Device:C_Polarized_Small
- added J1, J3: USB_A, Connector_USB:USB_A_Stewart_SS-52100-001_Horizontal, symbol Connector:USB_A
- added J2: HRO_TYPE-C-31-M-12, Connector_USB:USB_C_Receptacle_HRO_TYPE-C-31-M-12, symbol Connector:USB_C_Receptacle
- added R1, R2: 5.1k, Resistor_SMD:R_0805_2012Metric, symbol Device:R_Small
- added R10, R7, R8, R9: 10k, Resistor_SMD:R_0805_2012Metric, symbol Device:R_Small
- added R3, R4, R5, R6: 10K, Resistor_SMD:R_0805_2012Metric, symbol Device:R_Small
- added SW1: EN, Button_Switch_SMD:SW_SPST_EVPBF, symbol Switch:SW_Push
- added SW2: IO9, Button_Switch_SMD:SW_SPST_EVPBF, symbol Switch:SW_Push
- added U1, U2: AP22804AW5, Package_TO_SOT_SMD:SOT-23-5, symbol Power_Management:AP22804AW5
- added U3: ESP32-C3-WROOM-02-N4, MCU_Espressif_custom:MODULE_ESP32-C3-WROOM-02-H4, symbol MCU_Espressif_custom:ESP32-C3-WROOM-02-N4
- added U?: MCP1700T-3302E, Package_TO_SOT_SMD:SOT-23, symbol Regulator_Linear:MCP1700-3302E_SOT23
Connections:
- new net +3.3V: C1.1, C2.1, C?.1, R3.1, R4.1, R5.1, R6.1, U3.1 (3V3), U?.2 (VO)
- new net CC1: J2.A5 (CC1), R2.2
- new net CC2: J2.B5 (CC2), R1.2
- new net D+: J2.A6 (D+), J2.B6 (D+), U3.14 (IO19)
- new net D-: J2.A7 (D-), J2.B7 (D-), U3.13 (IO18)
- new net EN: C3.1, R3.2, SW1.2, U3.2 (EN)
- new net GND: C1.2, C10.1, C11.1, C2.2, C3.2, C4.2, C5.2, C6.1, C7.1, C8.2, C9.2, C?.2, C?.2, J1.4 (GND), J2.A1 (GND), J2.A12 (GND), J2.B1 (GND), J2.B12 (GND), J2.S1 (SHIELD), J3.4 (GND), R1.1, R10.2, R2.1, R8.2, SW1.1, SW2.1, U1.2 (GND), U2.2 (GND), U3.19 (GND), U3.20 (GND), U3.21 (GND), U3.22 (GND), U3.23 (GND), U3.24 (GND), U3.25 (GND), U3.26 (GND), U3.27 (GND), U3.28 (GND), U3.29 (GND), U3.30 (GND), U3.31 (GND), U3.32 (GND), U3.33 (GND), U3.34 (GND), U3.35 (GND), U3.36 (GND), U3.37 (GND), U3.38 (GND), U3.39 (GND), U3.9 (GND), U?.1 (GND)
- new net I010: R7.1, U1.3 (~{FLG}), U3.10 (IO10)
- new net IO2: R5.2, U3.16 (IO2)
- new net IO3: R10.1, U2.4 (EN), U3.15 (IO3)
- new net IO7: R8.1, U1.4 (EN), U3.6 (IO7)
- new net IO8: R6.2, U3.7 (IO8)
- new net IO9: R4.2, R9.1, SW2.2, U2.3 (~{FLG}), U3.8 (IO9)
- new net USB1_VCC: C4.1, C5.1, J1.1 (VBUS), U1.1 (OUT)
- new net USB2_VCC: C8.1, C9.1, J3.1 (VBUS), U2.1 (OUT)
- new net VCC: C10.2, C11.2, C6.2, C7.2, C?.1, J2.A4 (VBUS), J2.A9 (VBUS), J2.B4 (VBUS), J2.B9 (VBUS), R7.2, R9.2, U1.5 (IN), U2.5 (IN), U?.3 (VI)
- no-connect marks 0 -> 23
